File: KiCad_board/125khz_rfid_reader.kicad_pcb (KiCad board)
At the start: 2 copper layers, 49 x 71.5 mm, 36 parts, among them J1 SPI pins, J2 UART pins, Q1 STC945, Q4 BS170, Q5 2SC9014, SW1 Switch Mode, SW2 Save Mode, U1 LM358, U2 ATmega8A-A, U4 L78L05_TO92

Commit message: board added
Other:
- board text removed: "I have used vias as a placeholder for jump wires"
Changed lines of the file:
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@@
     (effects (font (size 1 1) (thickness 0.15)) (justify left bottom mirror))
-  )
-  (gr_text "I have used vias as a \nplaceholder for jump wires" (at 127.635 67.945) (layer "User.2")
-    (effects (font (size 3 3) (thickness 0.4)) (justify left bottom))
   )
   (segment (start 108.331 69.723) (end 106.934 71.12) (width 0.75) (layer "F.Cu") (net 1))
